File: Hardware/PCB.kicad_pcb (KiCad board)
At the start: 2 copper layers, 140 x 180 mm, 43 parts, among them J1 Conn_01x15, J2 Conn_01x15, J3 Conn_01x19, J4 Conn_01x19, Q5 NMOS, Q6 NMOS, Q7 NMOS, Q8 NMOS, U10 TLV379IDR, U11 LM7803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

Commit message: Save before using via-stiching script
Routing:
- net Net-(Q5-D): track 112.9 -> 114.3 mm
- net GND: track 221.0 -> 222.3 mm
Other:
- board text added: "--------------------- FALOWNIK --------------------- Autorzy projektu: Przemysław Lis Mateusz Kubsiewicz Jakub Banasiak Politechnka Wrocławska 2025"
- board text added: "{ "ViaStitching": "0.2", "GND": { "HSpacing": "1", "VSpacing": "1", "HOffset": "0", "VOffset": "0", "Clearance": "4", "Randomize": false } }"
- board text removed: "FALOWNIK Autorzy projektu: Przemysław Lis Mateusz Kubsiewicz Jakub Banasiak Politechnka Wrocławska 2025"
Changed lines of the file:
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@@
 		(tags "capacitor")
 		(property "Reference" "C17"
-			(at 0 -1.85 90)
+			(at 0.245 -2 90)
 			(layer "F.SilkS")
 			(effects
@@
 		(tags "capacitor")
 		(property "Reference" "C23"
-			(at 0 -1.85 90)
+			(at -2.995 0.5 180)
 			(layer "F.SilkS")
 			(effects
@@
 		(tags "resistor")
 		(property "Reference" "R13"
-			(at 0 -2.28 90)
+			(at -0.723737 2.4 90)
 			(layer "F.SilkS")
 			(effects
@@
 		(tags "Diode Mini-MELF (SOD-80)")
 		(property "Reference" "D6"
-			(at 0 -2 90)
+			(at -3.62 0.05 0)
 			(layer "F.SilkS")
 			(effects
@@
 	)
 	(gr_line
-		(start 189 188.68)
-		(end 187 186.68)
-		(stroke
-			(width 2)
-			(type solid)
-		)
-		(layer "F.Cu")
-		(net 9)
-	)
-	(gr_line
 		(start 194 174.68)
 		(end 162 147.68)
@@
 			(type solid)
 		)
-		(layer "F.Cu")
+		(layers "F.Cu" "F.Mask")
+		(solder_mask_margin 0.5)
 		(net 8)
 	)
 	(gr_rect
-		(start 150 85)
-		(end 290 265)
+		(start 138 86.6)
+		(end 278 266.6)
 		(stroke
 			(width 0.05)
@@
 		(layer "Edge.Cuts")
 	)
-	(gr_text "FALOWNIK\n\nAutorzy projektu:\nPrzemysław Lis\nMateusz Kubsiewicz\nJakub Banasiak\n\nPolitechnka Wrocławska 2025"
-		(at 215.6 242.2 0)
+	(gr_text "---------------------\nFALOWNIK\n---------------------\nAutorzy projektu:\nPrzemysław Lis\nMateusz Kubsiewicz\nJakub Banasiak\n\nPolitechnka Wrocławska 2025"
+		(at 209.6 240.4 0)
 		(layer "F.Cu")
 		(effects
@@
 		)
 	)
+	(gr_text "{\n  \"ViaStitching\": \"0.2\",\n  \"GND\": {\n    \"HSpacing\": \"1\",\n    \"VSpacing\": \"1\",\n    \"HOffset\": \"0\",\n    \"VOffset\": \"0\",\n    \"Clearance\": \"4\",\n    \"Randomize\": false\n  }\n}"
+		(at 0 0 0)
+		(layer "User.9")
+		(effects
+			(font
+				(size 1.27 1.27)
+			)
+			(justify left top)
+		)
+	)
 	(segment
 		(start 222 156.18)
@@
 	)
 	(segment
-		(start 235.700999 180.965371)
-		(end 235.700999 185.677471)
-		(width 1)
+		(start 229.438416 153.565824)
+		(end 226.885824 153.565824)
+		(width 0.5)
 		(layer "B.Cu")
 		(net 2)
 	)
 	(segment
-		(start 229.438416 153.565824)
-		(end 226.885824 153.565824)
-		(width 0.5)
+		(start 231.914628 177.179)
+		(end 236.4 181.664372)
+		(width 1)
 		(layer "B.Cu")
 		(net 2)
 	)
 	(segment
-		(start 235.700999 185.677471)
-		(end 228.19847 193.18)
+		(start 236.4 181.664372)
+		(end 236.4 186.05)
 		(width 1)
 		(layer "B.Cu")
@@
 	)
 	(segment
-		(start 230 178.18)
-		(end 231.001 177.179)
+		(start 231.001 177.179)
+		(end 231.914628 177.179)
 		(width 1)
 		(layer "B.Cu")
@@
 	)
 	(segment
-		(start 228.19847 193.18)
-		(end 225.1 193.18)
-		(width 1)
-		(layer "B.Cu")
-		(net 2)
-	)
-	(segment
-		(start 231.001 177.179)
-		(end 231.914628 177.179)
-		(width 1)
-		(layer "B.Cu")
-		(net 2)
-	)
-	(segment
-		(start 231.914628 177.179)
-		(end 235.700999 180.965371)
+		(start 236.4 165.18)
+		(end 231 165.18)
 		(width 1)
 		(layer "B.Cu")
@@
 	)
 	(segment
-		(start 236.4 165.18)
-		(end 231 165.18)
+		(start 236.4 186.05)
+		(end 229.27 193.18)
 		(width 1)
 		(layer "B.Cu")
@@
 	)
 	(segment
+		(start 230 178.18)
+		(end 231.001 177.179)
+		(width 1)
+		(layer "B.Cu")
+		(net 2)
+	)
+	(segment
 		(start 211.1 181.48)
 		(end 211.1 179.5)
@@
 	)
 	(segment
+		(start 229.27 193.18)
+		(end 225.1 193.18)
+		(width 1)
+		(layer "B.Cu")
+		(net 2)
+	)
+	(segment
 		(start 247.5 96.18)
 		(end 251.7 96.18)
@@
 	)
 	(segment
-		(start 190 189.68)
-		(end 190 189.7)
-		(width 2)
-		(layer "F.Cu")
-		(net 9)
-	)
-	(segment
 		(start 204.9 191.88)
 		(end 201.7 191.88)
@@
 	)
 	(segment
-		(start 201.7 191.88)
-		(end 201 191.18)
-		(width 0.5)
-		(layer "F.Cu")
-		(net 9)
-	)
-	(segment
-		(start 189 188.68)
-		(end 190 189.68)
-		(width 2)
-		(layer "F.Cu")
-		(net 9)
-	)
-	(segment
 		(start 190.48 190.18)
-		(end 191.75 190.18)
+		(end 178 177.7)
 		(width 2)
 		(layer "F.Cu")
@@
 	)
 	(segment
-		(start 201.1 193.38)
-		(end 201 193.48)
-		(width 0.5)
+		(start 190.48 190.18)
+		(end 191.75 190.18)
+		(width 2)
+		(layer "F.Cu")
+		(net 9)
+	)
+	(segment
+		(start 162 177.68)
+		(end 178 177.68)
+		(width 2)
 		(layer "F.Cu")
 		(net 9)
@@
 	)
 	(segment
-		(start 190 189.7)
-		(end 190.48 190.18)
+		(start 178 177.7)
+		(end 178 177.68)
 		(width 2)
 		(layer "F.Cu")
@@
 		(start 234.5 180.68)
 		(end 234.5 185.18)
-		(width 1)
-		(layer "F.Cu")
-		(net 9)
-	)
-	(segment
-		(start 178 177.68)
-		(end 187 186.68)
-		(width 2)
-		(layer "F.Cu")
-		(net 9)
-	)
-	(segment
-		(start 162 177.68)
-		(end 178 177.68)
-		(width 2)
+		(width 1.5)
 		(layer "F.Cu")
 		(net 9)
@@
 		(net 9)
 	)
-	(segment
-		(start 189 188.155)
-		(end 189 188.68)
-		(width 0.5)
-		(layer "F.Cu")
-		(net 9)
-	)
 	(via
-		(at 234.5 183.18)
+		(at 234.2 183.15)
 		(size 0.6)
 		(drill 0.3)
@@
 	)
 	(via
-		(at 234.5 185.18)
+		(at 234.2 185.15)
 		(size 0.6)
 		(drill 0.3)
@@
 	)
 	(via
-		(at 234.5 182.68)
+		(at 234.8 182.65)
 		(size 0.6)
 		(drill 0.3)
@@
 	)
 	(via
-		(at 234.5 184.68)
+		(at 234.8 184.65)
 		(size 0.6)
 		(drill 0.3)
@@
 	)
 	(via
-		(at 234.5 184.18)
+		(at 234.2 184.15)
 		(size 0.6)
 		(drill 0.3)
@@
 	)
 	(via
-		(at 234.5 183.68)
+		(at 234.8 183.65)
 		(size 0.6)
 		(drill 0.3)
@@
 	)
 	(segment
-		(start 234.5 184.68)
-		(end 234.5 184.18)
-		(width 1)
-		(layer "B.Cu")
-		(net 9)
-	)
-	(segment
 		(start 220 188.98)
 		(end 220 187.96)
@@
 	)
 	(segment
-		(start 234.5 183.18)
-		(end 234.5 182.68)
-		(width 1)
-		(layer "B.Cu")
-		(net 9)
-	)
-	(segment
-		(start 234.5 184.18)
-		(end 234.5 183.68)
-		(width 1)
-		(layer "B.Cu")
-		(net 9)
-	)
-	(segment
 		(start 218.6 190.38)
 		(end 220 188.98)
@@
 	(segment
 		(start 234.5 185.18)
-		(end 234.5 184.68)
-		(width 1)
-		(layer "B.Cu")
-		(net 9)
-	)
-	(segment
-		(start 234.5 183.68)
-		(end 234.5 183.18)
-		(width 1)
+		(end 234.5 182.4)
+		(width 1.5)
 		(layer "B.Cu")
 		(net 9)

Commit message: Run via stitching
Vias 1mm size/0.3mm, spacing 6x6mm, clearance 3mm
Routing:
- net GND: vias 24 -> 467
Other:
- board text added: "{ "ViaStitching": "0.2", "GND": { "HSpacing": "6", "VSpacing": "6", "HOffset": "0", "VOffset": "0", "Clearance": "3", "Randomize": false } }"
